Commit message: Replace complete urdf file
- Extracted and imported three links from main stl file
- Modified the coordinate frames of the links
- Located the links in the urdf file

TODO:
* STL file unit needs to be corrected
* urdf file should be modified to use args as parameters

File: src/cartesian_description/urdf/cartesian.urdf (robot description, URDF)
Before this commit: robot cartesian_robot, 4 links, 3 joints
Links:
- link link1: geometry collision mesh filename=package://cartesian_description/meshes/base_link.stl; visual mesh filename=package://cartesian_description/meshes/base_link.stl

Commit message: Cartesian_controller added.
    - Corrected urdf unit scale,
    - Added gazebo_plugins into the urdf file,
    - Added cartesian_crontroller so that the robot is ready to be simulate in gazebo.

    TODO:
    * use xacro in the urdf file,
    * correct the dynamic properties of the links and joints,
    * use cpr_robot along with cartesian_description

File: src/cartesian_description/urdf/cartesian.urdf (robot description, URDF)
Before this commit: robot cartesian_robot, 4 links, 3 joints
Links:
- link link1: mass 1 -> 0.6; geometry collision mesh filename=package://cartesian_description/meshes/base_link.stl scale=0.001 0.001 0.001; visual mesh filename=package://cartesian_description/meshes/base_link.stl scale=0.001 0.001 0.001
- link link2: mass 1 -> 0.3; geometry collision mesh filename=package://cartesian_description/meshes/link2.stl scale=0.001 0.001 0.001; visual mesh filename=package://cartesian_description/meshes/link2.stl scale=0.001 0.001 0.001
- link link3: mass 1 -> 0.100; geometry collision mesh filename=package://cartesian_description/meshes/link3.stl scale=0.001 0.001 0.001; visual mesh filename=package://cartesian_description/meshes/link3.stl scale=0.001 0.001 0.001
Joints:
- joint link1_link2: limit lower=-1 upper=1 effort=1000.0 velocity=0.5 -> lower=-10 upper=1000 effort=1000.0 velocity=0.5; origin xyz=0 0 0 -> xyz=0.120 0 0.055
- joint link2_link3: axis (none) -> 0 1 0; origin xyz=0 0 0 -> xyz=0 0.150 0.010
