Commit message: add third link. Loaded in rviz.

File: src/cartesian_description/urdf/cartesian_robot_simulation.urdf (robot description, URDF)
Before this commit: robot cartesian_robot, 4 links, 3 joints
Links:
- added link circular_link; collision mesh filename=package://cartesian_description/meshes/circular_link.stl scale=0.01 0.01 0.01; visual mesh filename=package://cartesian_description/meshes/circular_link.stl scale=0.01 0.01 0.01
Joints:
- added joint joint3: type revolute, parent link3, child circular_link, origin xyz=0.08 0.0 0.010, axis 0 0 1, limit lower=-1 upper=1 effort=1000.0 velocity=0.5

Commit message: Added third motor parts in the urdf file.

File: src/cartesian_description/urdf/cartesian_robot_simulation.urdf (robot description, URDF)
Before this commit: robot cartesian_robot, 5 links, 4 joints
Links:
- added link mounting_link, mass 0.100; collision mesh filename=package://cartesian_description/meshes/gearbasev1.stl scale=0.0254 0.0254 0.0254; visual mesh filename=package://cartesian_description/meshes/gearbasev1.stl scale=0.0254 0.0254 0.0254
- link circular_link: mass None -> 0.100; geometry collision mesh filename=package://cartesian_description/meshes/circular_link.stl scale=0.0254 0.0254 0.0254; visual mesh filename=package://cartesian_description/meshes/circular_link.stl scale=0.0254 0.0254 0.0254
Joints:
- added joint third_motor_mounting_joint: type fixed, parent link3, child mounting_link, origin xyz=0.0 0.0 0.0
- joint joint3: origin xyz=0.08 0.0 0.010 -> xyz=0.305 0.0 0.021; parent link3 -> mounting_link; type revolute -> continuous
