Commit message: Adopt cartesian_description pkg to work with both simulation and hardware runs

File: src/cartesian_description/urdf/cartesian_robot_hardware.urdf (robot description, URDF)
Before this commit: robot cartesian_robot, 4 links, 3 joints
Joints:
- removed joint link1_link2
- removed joint link2_link3
- added joint joint1: type prismatic, parent link1, child link2, origin xyz=0.120 0 0.055, limit lower=-10 upper=1000 effort=1000.0 velocity=0.5
- added joint joint2: type prismatic, parent link2, child link3, origin xyz=0 0.150 0.010, axis 0 1 0, limit lower=-1 upper=1 effort=1000.0 velocity=0.5

Commit message: Adopted all launch files to run under name_space
- rviz in simulation tested successfully.
- gazebo loading tested successfully.
- controllers for the cartesian tested successfully in gazebo.

File: src/cartesian_description/urdf/cartesian_robot_hardware.urdf (robot description, URDF)
Before this commit: robot cartesian_robot, 4 links, 3 joints
Links:
- added link circular_link, mass 0.100; collision mesh filename=package://cartesian_description/meshes/circular_link.stl scale=0.0254 0.0254 0.0254; visual mesh filename=package://cartesian_description/meshes/circular_link.stl scale=0.0254 0.0254 0.0254
- added link mounting_link, mass 0.100; collision mesh filename=package://cartesian_description/meshes/gearbasev1.stl scale=0.0254 0.0254 0.0254; visual mesh filename=package://cartesian_description/meshes/gearbasev1.stl scale=0.0254 0.0254 0.0254
Joints:
- added joint joint3: type continuous, parent mounting_link, child circular_link, origin xyz=0.305 0.0 0.021, axis 0 0 1, limit lower=-1 upper=1 effort=1000.0 velocity=0.5
- added joint third_motor_mounting_joint: type fixed, parent link3, child mounting_link, origin xyz=0.0 0.0 0.0

Commit message: commit tested changes to launch files. Added configuration .yaml file.

File: src/cartesian_description/urdf/cartesian_robot_hardware.urdf (robot description, URDF)
Before this commit: robot cartesian_, 6 links, 5 joints
Joints:
- joint joint1: limit lower=-10 upper=1000 effort=1000.0 velocity=0.5 -> lower=0 upper=1 effort=1000.0 velocity=0.5
